File: Electronics/laser_controller/laser_controller.kicad_pcb (KiCad board)
At the start: 2 copper layers, 100 x 80 mm, 47 parts, among them J1 Conn_01x02_Pin, J2 Conn_01x02_Pin, J3 Conn_01x02_Pin, J4 Conn_01x02_Pin, J5 Conn_01x02_Pin, J6 Conn_01x02_Pin, J7 Conn_01x02_Pin, J8 FTSH-105-01-F-DV-P-TR, J9 Conn_01x04_Pin, Q1 AO3400A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

Commit message: fixed too many bugs
Parts:
- removed J5, J6, J7: Conn_01x02_Pin, Connector_PinHeader_2.54mm:PinHeader_1x02_P2.54mm_Horizontal
- added C18: 100n, Capacitor_SMD:C_0805_2012Metric, F.Cu at (149.9, 106.4)
- added C19: 100n, Capacitor_SMD:C_0805_2012Metric, F.Cu at (138.5, 106.4)
- added D2: SM4007PL, Diode_SMD:D_SOD-123, F.Cu at (175.2, 127.1)
- added Q2: AO3400A, Package_TO_SOT_SMD:SOT-23, F.Cu at (176.8, 122.6)
- added R4: 10k, Resistor_SMD:R_0805_2012Metric, F.Cu at (176.8, 118.6)
- added U10: TXS0108EPW, Package_SO:Texas_PW0020A_TSSOP-20_4.4x6.5mm_P0.65mm, F.Cu at (144.1, 106.5)
- J1, J2, J3, J4: value Conn_01x02_Pin -> S3B-PH-K-S_LF__SN_; footprint Connector_PinHeader_2.54mm:PinHeader_1x02_P2.54mm_Horizontal -> Connector_JST:JST_PH_S3B-PH-K_1x03_P2.00mm_Horizontal
- moved J3 36.8 mm to (120.0, 132.0), turned to 0 degrees
- moved J8 33.6 mm to (152.3, 76.9)
- moved J2 29.4 mm to (135.0, 132.0), turned to 0 degrees
- moved J9 26.5 mm to (163.8, 114.0), turned to 0 degrees
- moved J1 25.6 mm to (150.0, 132.0), turned to 0 degrees
- moved J4 25.6 mm to (170.0, 132.2), turned to 0 degrees
- moved C10 7.84 mm to (128.1, 114.7), turned to 90 degrees
- moved Q1 7.60 mm to (167.8, 122.6)
- moved R3 7.60 mm to (167.8, 118.6)
- moved D1 6.33 mm to (169.4, 127.1)
- moved C7 5.65 mm to (111.9, 115.8)
- moved C9 5.65 mm to (111.8, 113.4)
- moved C14 5.57 mm to (150.0, 115.9)
- moved C15 5.57 mm to (150.0, 113.6)
- moved C11 4.49 mm to (130.5, 114.7), turned to 90 degrees
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Connections:
- D1 pad 2: Net-(D1-A) -> Motor- A
- J1 pad 1: +3.3V -> DAC_A1
- J1 pad 2: Net-(D1-A) -> GND
- J2 pad 1: GND -> DAC_B1
- J2 pad 2: DAC_A0 -> GND
- J3 pad 1: GND -> DAC_C1
- J3 pad 2: DAC_A1 -> GND
- J4 pad 1: GND -> Motor- A
- J4 pad 2: DAC_B0 -> +3.3V
- J9 pad 2: CLK -> CLK_B
- J9 pad 3: MOSI -> MOSI_B
- J9 pad 4: CS_A -> CS_A_B
- Q1 pad 3: Net-(D1-A) -> Motor- A
- U2 pad 11: unconnected-(U2-GP8-Pad11) -> OE
- U4 pad 3: CS_C -> CS_C_B
- U4 pad 4: CLK -> CLK_B
- U4 pad 5: MOSI -> MOSI_B
- U6 pad 3: CS_B -> CS_B_B
- U6 pad 4: CLK -> CLK_B
- U6 pad 5: MOSI -> MOSI_B
- U8 pad 3: CS_A -> CS_A_B
- U8 pad 4: CLK -> CLK_B
- U8 pad 5: MOSI -> MOSI_B
Routing:
- net CLK_B: track 0.00 -> 65.0 mm, vias 0 -> 4
- net MOSI_B: track 0.00 -> 62.9 mm, vias 0 -> 4
- net CLK: track 105.0 -> 53.5 mm, vias 4 -> 1
- net MOSI: track 102.6 -> 51.2 mm, vias 5 -> 1
- net OE: track 0.00 -> 39.1 mm
- net SWDIO: track 15.3 -> 52.0 mm, vias 0 -> 2
- net SWDCLK: track 25.2 -> 59.5 mm, vias 0 -> 2
- net CS_C_B: track 0.00 -> 33.6 mm
- net CS_A_B: track 0.00 -> 27.2 mm, vias 0 -> 4
- net SWO: track 68.8 -> 47.8 mm, vias 0 -> 2
- net CS_A: track 66.3 -> 47.1 mm, vias 3 -> 0
- net CS_B: track 61.5 -> 44.2 mm, vias 2 -> 0
- net CS_B_B: track 0.00 -> 13.6 mm
- net +2V5: track 78.5 -> 68.3 mm, vias 0 -> 4
- net Motor- B: track 0.00 -> 9.81 mm
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